Commit message: WIP,mechanical-confirm rviz loaded, bug: semi_sphere not display

File: mechanical/robot_model_try1/turtlebot3_harvest.urdf.xacro (robot description, xacro)
@@ -1,60 +1,45 @@
 <?xml version="1.0" ?>
 <robot name="turtlebot3_burger" xmlns:xacro="http://ros.org/wiki/xacro">
-  <xacro:include filename="$(find turtlebot3_description)/urdf/common_properties.xacro"/>
   <link name="base_footprint"/>
   <joint name="base_joint" type="fixed">
     <parent link="base_footprint"/>
     <child link="base_link"/>
-    <origin xyz="0.0 0.0 0.010" rpy="0 0 0"/>
+    <origin xyz="0.0 0.0 0" rpy="0 0 0"/>
   </joint>
   <link name="base_link">
     <visual>
-      <origin xyz="-0.032 0 0.0" rpy="0 0 0"/>
+      <origin xyz="0 0 0.0" rpy="0 0 0"/>
       <geometry>
-        <mesh filename="package://turtlebot3_description/meshes/bases/cyliner.stl" scale="0.001 0.001 0.001"/>
+        <mesh filename="package://turtlebot3_description/meshes/bases/cyliner.stl" scale="1 1 1"/>
       </geometry>
       <material name="light_black"/>
     </visual>
     <collision>
-      <origin xyz="-0.032 0 0.070" rpy="0 0 0"/>
+      <origin xyz="0 0 200" rpy="0 0 0"/>
       <geometry>
-        <box size="0.140 0.140 0.143"/>
+        <box size="100 100 200"/>
       </geometry>
     </collision>
-    <inertial>
-      <origin xyz="0 0 0" rpy="0 0 0"/>
-      <mass value="8.2573504e-01"/>
-      <inertia ixx="2.2124416e-03" ixy="-1.2294101e-05" ixz="3.4938785e-05"
-               iyy="2.1193702e-03" iyz="-5.0120904e-06"
-               izz="2.0064271e-03" />
-    </inertial>
   </link>
   <joint name="semi_sphere_joint" type="continuous">
     <parent link="base_link"/>
     <child link="semi_sphere_link"/>
-    <origin xyz="0.0 0.08 0.023" rpy="-1.57 0 0"/>
+    <origin xyz="0 0 200" rpy="0 0 1.57"/>
     <axis xyz="0 0 1"/>
   </joint>
   <link name="semi_sphere_link">
     <visual>
-      <origin xyz="0 0 0" rpy="1.57 0 0"/>
+      <origin xyz="0 0 200" rpy="0 0 1.57"/>
       <geometry>
-        <mesh filename="package://turtlebot3_description/meshes/bases/semi_sphere.stl" scale="0.001 0.001 0.001"/>
+        <mesh filename="package://turtlebot3_description/meshes/bases/semi_sphere.stl" scale="1 1 1"/>
       </geometry>
       <material name="dark"/>
     </visual>
     <collision>
-      <origin xyz="0 0 0" rpy="0 0 0"/>
+      <origin xyz="0 0 200" rpy="0 0 0"/>
       <geometry>
-        <cylinder length="0.018" radius="0.033"/>
+        <cylinder length="200" radius="50"/>
       </geometry>
     </collision>
-    <inertial>
-      <origin xyz="0 0 0" />
-      <mass value="2.8498940e-02" />
-      <inertia ixx="1.1175580e-05" ixy="-4.2369783e-11" ixz="-5.9381719e-09"
-               iyy="1.1192413e-05" iyz="-1.4400107e-11"
-               izz="2.0712558e-05" />
-      </inertial>
   </link>
 </robot>

Commit message: WIP:mechanical-saw 2 STL by fixed joint, revised position

File: mechanical/robot_model_try1/turtlebot3_harvest.urdf.xacro (robot description, xacro)
@@ -22,13 +22,13 @@
     </collision>
   </link>
-  <joint name="semi_sphere_joint" type="continuous">
+  <joint name="semi_sphere_joint" type="fixed">
     <parent link="base_link"/>
     <child link="semi_sphere_link"/>
-    <origin xyz="0 0 200" rpy="0 0 1.57"/>
+    <origin xyz="0 0 10" rpy="0 0 1.57"/>
     <axis xyz="0 0 1"/>
   </joint>
   <link name="semi_sphere_link">
     <visual>
-      <origin xyz="0 0 200" rpy="0 0 1.57"/>
+      <origin xyz="0 0 10" rpy="0 0 1.57"/>
       <geometry>
         <mesh filename="package://turtlebot3_description/meshes/bases/semi_sphere.stl" scale="1 1 1"/>
@@ -37,7 +37,7 @@
     </visual>
     <collision>
-      <origin xyz="0 0 200" rpy="0 0 0"/>
+      <origin xyz="0 0 10" rpy="0 0 0"/>
       <geometry>
-        <cylinder length="200" radius="50"/>
+        <cylinder length="10" radius="5"/>
       </geometry>
     </collision>
